File: prj-kicad/carinsitu-power.sch (KiCad schematic (older format))
At the start: 0 parts

Commit message: = ADD: insert a 3V3 power regulator. Schematic and place ok, routing not complete
Parts:
- added C6, C7: C, carinsitu:SMD0805, symbol C
- added C8: C, carinsitu:SMD1210, symbol C
- added L2: FB600, carinsitu:SMD0603, symbol INDUCTOR
- added L3: 4,7uH, carinsitu:I_TYS4012, symbol INDUCTOR
- added R6: 150k, carinsitu:SMD0603, symbol R
- added R7: 48,7k, carinsitu:SMD0603, symbol R
- added TP1: CONN_1, symbol CONN_1
- added U6: TPS560200, carinsitu:SOT23-6, symbol TPS560200
Connections:
- new net: TP1.1, U6.1 (EN)
- new net: L3.1, U6.3 (PH)
- new net: C7.1, L2.2, U6.4 (VIN)
- new net: R6.2, R7.1, U6.5 (FB)
- new net +3V3: C8.1, L3.2, R6.1
- new net +VBAT: C6.1, L2.1
- new net GND: C6.2, C7.2, C8.2, R7.2, U6.2
Changed lines of the file:
@@
 EESchema Schematic File Version 2
 LIBS:carinsitu
+LIBS:nauticsafe-gateway
 LIBS:carinsitu-cache
 EELAYER 25 0
@@
 $Descr A4 11693 8268
 encoding utf-8
-Sheet 1 1
+Sheet 2 2
 Title ""
 Date ""
@@
 Comment4 ""
 $EndDescr
+$Comp
+L TPS560200 U6
+U 1 1 5D25329E
+P 5650 1450
+F 0 "U6" H 5650 1850 60  0000 C CNN
+F 1 "TPS560200" H 5650 1450 60  0000 C CNN
+F 2 "carinsitu:SOT23-6" H 5650 1450 60  0001 C CNN
+F 3 "" H 5650 1450 60  0000 C CNN
+	1    5650 1450
+	1    0    0    -1
+$EndComp
+$Comp
+L CONN_1 TP1
+U 1 1 5D25331A
+P 5000 1850
+F 0 "TP1" H 5080 1850 40  0000 L CNN
+F 1 "CONN_1" H 5000 1905 30  0001 C CNN
+F 2 "" H 5000 1850 60  0001 C CNN
+F 3 "" H 5000 1850 60  0000 C CNN
+	1    5000 1850
+	0    1    1    0
+$EndComp
+Wire Wire Line
+	5000 1700 5000 1600
+Wire Wire Line
+	5000 1600 5100 1600
+$Comp
+L GND #PWR042
+U 1 1 5D25336A
+P 5650 1950
+F 0 "#PWR042" H 5650 1950 30  0001 C CNN
+F 1 "GND" H 5650 1880 30  0001 C CNN
+F 2 "" H 5650 1950 60  0000 C CNN
+F 3 "" H 5650 1950 60  0000 C CNN
+	1    5650 1950
+	1    0    0    -1
+$EndComp
+Wire Wire Line
+	5650 1950 5650 1900
+$Comp
+L C C7
+U 1 1 5D25338F
+P 4700 1600
+F 0 "C7" H 4750 1700 50  0000 L CNN
+F 1 "C" H 4750 1500 50  0000 L CNN
+F 2 "carinsitu:SMD0805" H 4700 1600 60  0001 C CNN
+F 3 "" H 4700 1600 60  0000 C CNN
+	1    4700 1600
+	1    0    0    -1
+$EndComp
+$Comp
+L GND #PWR043
+U 1 1 5D2533E0
+P 4700 1900
+F 0 "#PWR043" H 4700 1900 30  0001 C CNN
+F 1 "GND" H 4700 1830 30  0001 C CNN
+F 2 "" H 4700 1900 60  0000 C CNN
+F 3 "" H 4700 1900 60  0000 C CNN
+	1    4700 1900
+	1    0    0    -1
+$EndComp
+Wire Wire Line
+	4700 1900 4700 1800
+Wire Wire Line
+	4700 1400 4700 1300
+$Comp
+L +VBAT #PWR044
+U 1 1 5D253412
+P 3700 1200
+F 0 "#PWR044" H 3700 1160 30  0001 C CNN
+F 1 "+VBAT" H 3700 1310 30  0000 C CNN
+F 2 "" H 3700 1200 60  0000 C CNN
+F 3 "" H 3700 1200 60  0000 C CNN
+	1    3700 1200
+	1    0    0    -1
+$EndComp
+$Comp
+L C C6
+U 1 1 5D25343F
+P 3900 1600
+F 0 "C6" H 3950 1700 50  0000 L CNN
+F 1 "C" H 3950 1500 50  0000 L CNN
+F 2 "carinsitu:SMD0805" H 3900 1600 60  0001 C CNN
+F 3 "" H 3900 1600 60  0000 C CNN
+	1    3900 1600
+	1    0    0    -1
+$EndComp
+$Comp
+L GND #PWR045
+U 1 1 5D253472
+P 3900 1900
+F 0 "#PWR045" H 3900 1900 30  0001 C CNN
+F 1 "GND" H 3900 1830 30  0001 C CNN
+F 2 "" H 3900 1900 60  0000 C CNN
+F 3 "" H 3900 1900 60  0000 C CNN
+	1    3900 1900
+	1    0    0    -1
+$EndComp
+Wire Wire Line
+	3900 1900 3900 1800
+Wire Wire Line
+	3900 1400 3900 1300
+Connection ~ 4700 1300
+Wire Wire Line
+	3700 1200 3700 1300
+Connection ~ 3900 1300
+$Comp
+L INDUCTOR L2
+U 1 1 5D253528
+P 4300 1300
+F 0 "L2" V 4400 1300 60  0000 C CNN
+F 1 "FB600" V 4250 1300 40  0000 C CNN
+F 2 "carinsitu:SMD0603" H 4300 1300 60  0001 C CNN
+F 3 "" H 4300 1300 60  0000 C CNN
+	1    4300 1300
+	0    -1   -1   0
+$EndComp
+Wire Wire Line
+	3700 1300 4000 1300
+Wire Wire Line
+	4600 1300 5100 1300
+$Comp
+L INDUCTOR L3
+U 1 1 5D2537AF
+P 6600 1300
+F 0 "L3" V 6750 1300 60  0000 C CNN
+F 1 "4,7uH" V 6550 1300 40  0000 C CNN
+F 2 "carinsitu:I_TYS4012" H 6600 1300 60  0001 C CNN
+F 3 "" H 6600 1300 60  0000 C CNN
+	1    6600 1300
+	0    -1   -1   0
+$EndComp
+Wire Wire Line
+	6200 1300 6300 1300
+$Comp
+L R R6
+U 1 1 5D2538F4
+P 7000 1650
+F 0 "R6" V 7100 1650 50  0000 C CNN
+F 1 "150k" V 7000 1650 45  0000 C CNN
+F 2 "carinsitu:SMD0603" H 7000 1650 60  0001 C CNN
+F 3 "" H 7000 1650 60  0000 C CNN
+	1    7000 1650
+	1    0    0    -1
+$EndComp
+$Comp
+L R R7
+U 1 1 5D253941
+P 7000 2250
+F 0 "R7" V 7100 2250 50  0000 C CNN
+F 1 "48,7k" V 7000 2250 45  0000 C CNN
+F 2 "carinsitu:SMD0603" H 7000 2250 60  0001 C CNN
+F 3 "" H 7000 2250 60  0000 C CNN
+	1    7000 2250
+	1    0    0    -1
+$EndComp
+Wire Wire Line
+	7000 2000 7000 1900
+Wire Wire Line
+	7000 1950 6600 1950
+Wire Wire Line
+	6600 1950 6600 1600
+Wire Wire Line
+	6600 1600 6200 1600
+Connection ~ 7000 1950
+Wire Wire Line
+	7000 1400 7000 1300
+Wire Wire Line
+	6900 1300 7500 1300
+$Comp
+L GND #PWR046
+U 1 1 5D253A80
+P 7000 2550
+F 0 "#PWR046" H 7000 2550 30  0001 C CNN
+F 1 "GND" H 7000 2480 30  0001 C CNN
+F 2 "" H 7000 2550 60  0000 C CNN
+F 3 "" H 7000 2550 60  0000 C CNN
+	1    7000 2550
+	1    0    0    -1
+$EndComp
+Wire Wire Line
+	7000 2550 7000 2500
+$Comp
+L C C8
+U 1 1 5D253AC2
+P 7300 1650
+F 0 "C8" H 7350 1750 50  0000 L CNN
+F 1 "C" H 7350 1550 50  0000 L CNN
+F 2 "carinsitu:SMD1210" H 7300 1650 60  0001 C CNN
+F 3 "" H 7300 1650 60  0000 C CNN
+	1    7300 1650
+	1    0    0    -1
+$EndComp
+$Comp
+L GND #PWR047
+U 1 1 5D253B09
+P 7300 1900
+F 0 "#PWR047" H 7300 1900 30  0001 C CNN
+F 1 "GND" H 7300 1830 30  0001 C CNN
+F 2 "" H 7300 1900 60  0000 C CNN
+F 3 "" H 7300 1900 60  0000 C CNN
+	1    7300 1900
+	1    0    0    -1
+$EndComp
+Wire Wire Line
+	7300 1900 7300 1850
+Wire Wire Line
+	7300 1300 7300 1450
+Connection ~ 7000 1300
+$Comp
+L +3V3 #PWR048
+U 1 1 5D253B71
+P 7500 1200
+F 0 "#PWR048" H 7500 1160 30  0001 C CNN
+F 1 "+3V3" H 7500 1310 30  0000 C CNN
+F 2 "" H 7500 1200 60  0000 C CNN
+F 3 "" H 7500 1200 60  0000 C CNN
+	1    7500 1200
+	1    0    0    -1
+$EndComp
+Wire Wire Line
+	7500 1300 7500 1200
+Connection ~ 7300 1300
 $EndSCHEMATC

Commit message: = UPD: Replace ESP32 with ESP82xx to fit software requirements
Parts:
- renumbered L2 to L1, L3 to L2
Changed lines of the file:
@@
 	5000 1600 5100 1600
 $Comp
-L GND #PWR049
+L GND #PWR048
 U 1 1 5D25336A
 P 5650 1950
-F 0 "#PWR049" H 5650 1950 30  0001 C CNN
+F 0 "#PWR048" H 5650 1950 30  0001 C CNN
 F 1 "GND" H 5650 1880 30  0001 C CNN
 F 2 "" H 5650 1950 60  0000 C CNN
@@
 $EndComp
 $Comp
-L GND #PWR050
+L GND #PWR049
 U 1 1 5D2533E0
 P 4700 1900
-F 0 "#PWR050" H 4700 1900 30  0001 C CNN
+F 0 "#PWR049" H 4700 1900 30  0001 C CNN
 F 1 "GND" H 4700 1830 30  0001 C CNN
 F 2 "" H 4700 1900 60  0000 C CNN
@@
 	4700 1400 4700 1300
 $Comp
-L +VBAT #PWR051
+L +VBAT #PWR050
 U 1 1 5D253412
 P 3700 1200
-F 0 "#PWR051" H 3700 1160 30  0001 C CNN
+F 0 "#PWR050" H 3700 1160 30  0001 C CNN
 F 1 "+VBAT" H 3700 1310 30  0000 C CNN
 F 2 "" H 3700 1200 60  0000 C CNN
@@
 $EndComp
 $Comp
-L GND #PWR052
+L GND #PWR051
 U 1 1 5D253472
 P 3900 1900
-F 0 "#PWR052" H 3900 1900 30  0001 C CNN
+F 0 "#PWR051" H 3900 1900 30  0001 C CNN
 F 1 "GND" H 3900 1830 30  0001 C CNN
 F 2 "" H 3900 1900 60  0000 C CNN
@@
 Connection ~ 3900 1300
 $Comp
-L INDUCTOR L2
+L INDUCTOR L1
 U 1 1 5D253528
 P 4300 1300
-F 0 "L2" V 4400 1300 60  0000 C CNN
+F 0 "L1" V 4400 1300 60  0000 C CNN
 F 1 "FB600" V 4250 1300 40  0000 C CNN
 F 2 "carinsitu:SMD0603" H 4300 1300 60  0001 C CNN
@@
 	4600 1300 5100 1300
 $Comp
-L INDUCTOR L3
+L INDUCTOR L2
 U 1 1 5D2537AF
 P 6600 1300
-F 0 "L3" V 6750 1300 60  0000 C CNN
+F 0 "L2" V 6750 1300 60  0000 C CNN
 F 1 "4,7uH" V 6550 1300 40  0000 C CNN
 F 2 "carinsitu:I_TYS4012" H 6600 1300 60  0001 C CNN
@@
 	6900 1300 7500 1300
 $Comp
-L GND #PWR053
+L GND #PWR052
 U 1 1 5D253A80
 P 7000 2550
-F 0 "#PWR053" H 7000 2550 30  0001 C CNN
+F 0 "#PWR052" H 7000 2550 30  0001 C CNN
 F 1 "GND" H 7000 2480 30  0001 C CNN
 F 2 "" H 7000 2550 60  0000 C CNN
@@
 $EndComp
 $Comp
-L GND #PWR054
+L GND #PWR053
 U 1 1 5D253B09
 P 7300 1900
-F 0 "#PWR054" H 7300 1900 30  0001 C CNN
+F 0 "#PWR053" H 7300 1900 30  0001 C CNN
 F 1 "GND" H 7300 1830 30  0001 C CNN
 F 2 "" H 7300 1900 60  0000 C CNN
@@
 Connection ~ 7000 1300
 $Comp
-L +3V3 #PWR055
+L +3V3 #PWR054
 U 1 1 5D253B71
 P 7500 1200
-F 0 "#PWR055" H 7500 1160 30  0001 C CNN
+F 0 "#PWR054" H 7500 1160 30  0001 C CNN
 F 1 "+3V3" H 7500 1310 30  0000 C CNN
 F 2 "" H 7500 1200 60  0000 C CNN

Commit message: = UPD: Improve ESP82xx routing, connect main IOs (leds, esc, servo, ...)
Parts:
- TP1: footprint (none) -> carinsitu:TP_SMD
Changed lines of the file:
@@
 F 0 "TP1" H 5080 1850 40  0000 L CNN
 F 1 "CONN_1" H 5000 1905 30  0001 C CNN
-F 2 "" H 5000 1850 60  0001 C CNN
+F 2 "carinsitu:TP_SMD" H 5000 1850 60  0001 C CNN
 F 3 "" H 5000 1850 60  0000 C CNN
 	1    5000 1850
@@
 	5000 1600 5100 1600
 $Comp
-L GND #PWR048
+L GND #PWR050
 U 1 1 5D25336A
 P 5650 1950
-F 0 "#PWR048" H 5650 1950 30  0001 C CNN
+F 0 "#PWR050" H 5650 1950 30  0001 C CNN
 F 1 "GND" H 5650 1880 30  0001 C CNN
 F 2 "" H 5650 1950 60  0000 C CNN
@@
 $EndComp
 $Comp
-L GND #PWR049
+L GND #PWR051
 U 1 1 5D2533E0
 P 4700 1900
-F 0 "#PWR049" H 4700 1900 30  0001 C CNN
+F 0 "#PWR051" H 4700 1900 30  0001 C CNN
 F 1 "GND" H 4700 1830 30  0001 C CNN
 F 2 "" H 4700 1900 60  0000 C CNN
@@
 	4700 1400 4700 1300
 $Comp
-L +VBAT #PWR050
+L +VBAT #PWR052
 U 1 1 5D253412
 P 3700 1200
-F 0 "#PWR050" H 3700 1160 30  0001 C CNN
+F 0 "#PWR052" H 3700 1160 30  0001 C CNN
 F 1 "+VBAT" H 3700 1310 30  0000 C CNN
 F 2 "" H 3700 1200 60  0000 C CNN
@@
 $EndComp
 $Comp
-L GND #PWR051
+L GND #PWR053
 U 1 1 5D253472
 P 3900 1900
-F 0 "#PWR051" H 3900 1900 30  0001 C CNN
+F 0 "#PWR053" H 3900 1900 30  0001 C CNN
 F 1 "GND" H 3900 1830 30  0001 C CNN
 F 2 "" H 3900 1900 60  0000 C CNN
@@
 	6900 1300 7500 1300
 $Comp
-L GND #PWR052
+L GND #PWR054
 U 1 1 5D253A80
 P 7000 2550
-F 0 "#PWR052" H 7000 2550 30  0001 C CNN
+F 0 "#PWR054" H 7000 2550 30  0001 C CNN
 F 1 "GND" H 7000 2480 30  0001 C CNN
 F 2 "" H 7000 2550 60  0000 C CNN
@@
 $EndComp
 $Comp
-L GND #PWR053
+L GND #PWR055
 U 1 1 5D253B09
 P 7300 1900
-F 0 "#PWR053" H 7300 1900 30  0001 C CNN
+F 0 "#PWR055" H 7300 1900 30  0001 C CNN
 F 1 "GND" H 7300 1830 30  0001 C CNN
 F 2 "" H 7300 1900 60  0000 C CNN
@@
 Connection ~ 7000 1300
 $Comp
-L +3V3 #PWR054
+L +3V3 #PWR056
 U 1 1 5D253B71
 P 7500 1200
-F 0 "#PWR054" H 7500 1160 30  0001 C CNN
+F 0 "#PWR056" H 7500 1160 30  0001 C CNN
 F 1 "+3V3" H 7500 1310 30  0000 C CNN
 F 2 "" H 7500 1200 60  0000 C CNN

Commit message: = UPD: Improve power, fix 3V3 reg footprint and add routing
Parts:
- L1: footprint carinsitu:SMD0603 -> carinsitu:SMD0805
- U6: footprint carinsitu:SOT23-6 -> carinsitu:SOT23-5
Connections:
- net 3V3_SW: now reaches L2.1, U6.3 (PH)
Changed lines of the file:
@@
 F 0 "U6" H 5650 1850 60  0000 C CNN
 F 1 "TPS560200" H 5650 1450 60  0000 C CNN
-F 2 "carinsitu:SOT23-6" H 5650 1450 60  0001 C CNN
+F 2 "carinsitu:SOT23-5" H 5650 1450 60  0001 C CNN
 F 3 "" H 5650 1450 60  0000 C CNN
 	1    5650 1450
@@
 	5000 1600 5100 1600
 $Comp
-L GND #PWR063
+L GND #PWR064
 U 1 1 5D25336A
 P 5650 1950
-F 0 "#PWR063" H 5650 1950 30  0001 C CNN
+F 0 "#PWR064" H 5650 1950 30  0001 C CNN
 F 1 "GND" H 5650 1880 30  0001 C CNN
 F 2 "" H 5650 1950 60  0000 C CNN
@@
 $EndComp
 $Comp
-L GND #PWR064
+L GND #PWR065
 U 1 1 5D2533E0
 P 4700 1900
-F 0 "#PWR064" H 4700 1900 30  0001 C CNN
+F 0 "#PWR065" H 4700 1900 30  0001 C CNN
 F 1 "GND" H 4700 1830 30  0001 C CNN
 F 2 "" H 4700 1900 60  0000 C CNN
@@
 	4700 1400 4700 1300
 $Comp
-L +VBAT #PWR065
+L +VBAT #PWR066
 U 1 1 5D253412
 P 3700 1200
-F 0 "#PWR065" H 3700 1160 30  0001 C CNN
+F 0 "#PWR066" H 3700 1160 30  0001 C CNN
 F 1 "+VBAT" H 3700 1310 30  0000 C CNN
 F 2 "" H 3700 1200 60  0000 C CNN
@@
 $EndComp
 $Comp
-L GND #PWR066
+L GND #PWR067
 U 1 1 5D253472
 P 3900 1900
-F 0 "#PWR066" H 3900 1900 30  0001 C CNN
+F 0 "#PWR067" H 3900 1900 30  0001 C CNN
 F 1 "GND" H 3900 1830 30  0001 C CNN
 F 2 "" H 3900 1900 60  0000 C CNN
@@
 F 0 "L1" V 4400 1300 60  0000 C CNN
 F 1 "FB600" V 4250 1300 40  0000 C CNN
-F 2 "carinsitu:SMD0603" H 4300 1300 60  0001 C CNN
+F 2 "carinsitu:SMD0805" H 4300 1300 60  0001 C CNN
 F 3 "" H 4300 1300 60  0000 C CNN
 	1    4300 1300
@@
 	6900 1300 7500 1300
 $Comp
-L GND #PWR067
+L GND #PWR068
 U 1 1 5D253A80
 P 7000 2550
-F 0 "#PWR067" H 7000 2550 30  0001 C CNN
+F 0 "#PWR068" H 7000 2550 30  0001 C CNN
 F 1 "GND" H 7000 2480 30  0001 C CNN
 F 2 "" H 7000 2550 60  0000 C CNN
@@
 $EndComp
 $Comp
-L GND #PWR068
+L GND #PWR069
 U 1 1 5D253B09
 P 7300 1900
-F 0 "#PWR068" H 7300 1900 30  0001 C CNN
+F 0 "#PWR069" H 7300 1900 30  0001 C CNN
 F 1 "GND" H 7300 1830 30  0001 C CNN
 F 2 "" H 7300 1900 60  0000 C CNN
@@
 Connection ~ 7000 1300
 $Comp
-L +3V3 #PWR069
+L +3V3 #PWR070
 U 1 1 5D253B71
 P 7500 1200
-F 0 "#PWR069" H 7500 1160 30  0001 C CNN
+F 0 "#PWR070" H 7500 1160 30  0001 C CNN
 F 1 "+3V3" H 7500 1310 30  0000 C CNN
 F 2 "" H 7500 1200 60  0000 C CNN
@@
 	7500 1300 7500 1200
 Connection ~ 7300 1300
+Text Label 6200 1300 0    30   ~ 0
+3V3_SW
 $EndSCHEMATC
