File: prj-kicad/Power.kicad_sch (KiCad schematic)
At the start: 14 parts, among them P1 BAT, Q1 TJ15P04M3, SW1 SWITCH_SLIDE, U3 MAX17261xxTD

Commit message: schematic corrections and first PCB update
Connections:
- net +3V3: now also U3.1 (TH)
- net GNDD: now also U3.12 (ALRT)
- no-connect marks 4 -> 2
Changed lines of the file:
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@@
   (junction (at 199.39 74.93) (diameter 0) (color 0 0 0 0)
+  )
+  (junction (at 199.39 81.28) (diameter 0) (color 0 0 0 0)
   )
   (junction (at 100.33 100.33) (diameter 0) (color 0 0 0 0)
@@
   (no_connect (at 189.23 86.36))
   (no_connect (at 90.17 86.36))
-  (no_connect (at 209.55 91.44))
-  (no_connect (at 189.23 93.98))
   (wire (pts (xy 156.21 106.68) (xy 176.53 106.68))
     (stroke (width 0) (type default) (color 0 0 0 0))
@@
     (stroke (width 0) (type default) (color 0 0 0 0))
   )
+  (wire (pts (xy 215.9 91.44) (xy 215.9 92.71))
+    (stroke (width 0) (type default) (color 0 0 0 0))
+  )
   (wire (pts (xy 113.03 94.615) (xy 100.33 94.615))
     (stroke (width 0) (type default) (color 0 0 0 0))
@@
     (stroke (width 0) (type default) (color 0 0 0 0))
   )
+  (wire (pts (xy 209.55 91.44) (xy 215.9 91.44))
+    (stroke (width 0) (type default) (color 0 0 0 0))
+  )
   (wire (pts (xy 199.39 71.12) (xy 199.39 74.93))
     (stroke (width 0) (type default) (color 0 0 0 0))
@@
     (stroke (width 0) (type default) (color 0 0 0 0))
   )
+  (wire (pts (xy 185.42 81.28) (xy 199.39 81.28))
+    (stroke (width 0) (type default) (color 0 0 0 0))
+  )
+  (wire (pts (xy 189.23 93.98) (xy 185.42 93.98))
+    (stroke (width 0) (type default) (color 0 0 0 0))
+  )
   (wire (pts (xy 182.88 99.06) (xy 189.23 99.06))
     (stroke (width 0) (type default) (color 0 0 0 0))
@@
   )
   (wire (pts (xy 189.23 101.6) (xy 189.23 106.68))
+    (stroke (width 0) (type default) (color 0 0 0 0))
+  )
+  (wire (pts (xy 185.42 93.98) (xy 185.42 81.28))
     (stroke (width 0) (type default) (color 0 0 0 0))
   )
@@
     (pin "9")
   )
+  (symbol (lib_id "power:GNDD") (at 215.9 92.71 0) (unit 1)
+    (in_bom yes) (on_board yes) (fields_autoplaced)
+    (property "Reference" "#PWR?" (id 0) (at 215.9 99.06 0)
+      (effects (font (size 1.27 1.27)) hide)
+    )
+    (property "Value" "GNDD" (id 1) (at 215.9 97.79 0))
+    (property "Footprint" "" (id 2) (at 215.9 92.71 0)
+      (effects (font (size 1.27 1.27)) hide)
+    )
+    (property "Datasheet" "" (id 3) (at 215.9 92.71 0)
+      (effects (font (size 1.27 1.27)) hide)
+    )
+    (pin "1")
+  )
 )

Commit message: pcb update -wip-
Parts:
- renumbered R3 to R4
Changed lines of the file:
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@@
   (symbol (lib_id "carinsitu:R") (at 116.84 100.33 90) (unit 1)
     (in_bom yes) (on_board yes)
-    (property "Reference" "R3" (id 0) (at 116.84 102.87 90))
+    (property "Reference" "R4" (id 0) (at 116.84 102.87 90))
     (property "Value" "1k" (id 1) (at 116.84 100.33 90))
     (property "Footprint" "Resistor_SMD:R_0805_2012Metric" (id 2) (at 116.84 100.33 0)
